Commit message: modified:   diffdrive_bot/CMakeLists.txt 	new file:   diffdrive_bot/bringup/config/mapper_params_online_async.yaml 	modified:   diffdrive_bot/bringup/config/mira_controller.yaml 	new file:   diffdrive_bot/bringup/launch/custom_cartographer.launch.py 	modified:   diffdrive_bot/bringup/launch/diffbot.launch.py 	new file:   diffdrive_bot/bringup/launch/gazebo.launch.py 	modified:   diffdrive_bot/bringup/launch/gazebo_display.launch.xml 	new file:   diffdrive_bot/bringup/launch/robot_state_publsiher.xml 	new file:   diffdrive_bot/bringup/launch/rviz.launch.xml 	new file:   diffdrive_bot/bringup/worlds/maze.world 	new file:   diffdrive_bot/description/rviz/mira.rviz 	new file:   diffdrive_bot/description/rviz/rviz_config.rviz 	modified:   diffdrive_bot/description/urdf/common_properties.xacro 	new file:   diffdrive_bot/description/urdf/lidar.xacro 	modified:   diffdrive_bot/description/urdf/mira.urdf.xacro 	modified:   diffdrive_bot/description/urdf/mira_base.xacro 	new file:   diffdrive_bot/description/urdf/mira_gazebo.urdf.xacro 	modified:   diffdrive_bot/description/urdf/mira_gazebo.xacro 	modified:   diffdrive_bot/package.xml 	new file:   sensor_manip/CMakeLists.txt 	new file:   sensor_manip/package.xml 	new file:   sensor_manip/src/scan_update.cpp

File: diffdrive_bot/description/urdf/common_properties.xacro (robot description, xacro)
@@ -14,4 +14,7 @@
     <material name="yellow">
         <color rgba="1 1 0 1" />
+    </material>
+    <material name="red">
+        <color rgba="1 0 0 1"/>
     </material>
     <xacro:macro name="box_inertia" params="m l w h xyz rpy">

File: diffdrive_bot/description/urdf/mira_base.xacro (robot description, xacro)
@@ -7,6 +7,13 @@
     <xacro:property name="wheel_length" value="0.05" />
     <xacro:property name="caster_wheel_radius" value="${wheel_radius / 2.0}" />
-    <link name="base_footprint" />
-    <link name="base_link">
+    <link name="base_link" />
+    <link name="base_footprint">
+    </link>
+    <joint name="base_footprint_joint" type="fixed">
+        <parent link="base_link"/>
+        <child link="base_footprint"/>
+        <origin xyz="0 0 0" rpy="0 0 0"/>
+    </joint>
+    <link name="chassis">
         <visual>
             <geometry>
@@ -24,4 +31,21 @@
         <xacro:box_inertia m="5.0" l="${2*base_length}" w="${2*base_width}" h="${2*base_height}"
                            xyz="0 0 ${base_height / 2.0}" rpy="0 0 0" />
+    </link>
+    <link name="laser_base_link">
+        <visual>
+            <geometry>
+                <cylinder radius="0.05" length="0.05" />
+            </geometry>
+            <origin xyz="0 0 0.025" rpy="0 0 0" />
+            <material name="blue" />
+        </visual>
+        <collision>
+            <geometry>
+                <cylinder radius="0.05" length="0.05" />
+            </geometry>
+            <origin xyz="0 0 0.025" rpy="0 0 0" />
+            <xacro:cylinder_inertia m="0.1" r="0.05" l="0.1"
+                                    xyz="0 0 0" rpy="${pi / 2.0} 0 0" />
+        </collision>
     </link>
     <xacro:macro name="wheel_link" params="prefix">
@@ -63,11 +87,59 @@
                               xyz="0 0 0" rpy="0 0 0" />
     </link>
+    <xacro:macro name="support_link" params="suffix">
+        <link name="support_${suffix}">
+            <visual>
+                <geometry>
+                    <box size="0.05 0.05 0.2" />
+                </geometry>
+                <origin xyz="0 0 0.1" rpy="0 0 0" />
+                <material name="blue" />
+            </visual>
+            <collision>
+                <geometry>
+                    <box size="0.05 0.05 0.2" />
+                </geometry>
+                <origin xyz="0 0 0.1" rpy="0 0 0" />
+            </collision>
+            <xacro:box_inertia m="1.0" l="${2*0.05}" w="${2*0.05}" h="${2*0.2}"
+                            xyz="0 0 0.1" rpy="0 0 0" />
+        </link>
+    </xacro:macro>
+    <xacro:support_link suffix = "1"/>
+    <joint name="chassis_support_1" type="fixed">
+            <parent link="chassis"/>
+            <child link="support_1"/>
+            <origin xyz=" ${0.3 - (0.05/2.0)} ${0.2 - (0.05/2.0)} 0.2" rpy="0 0 0"/>
+    </joint>
+    <xacro:support_link suffix = "2"/>
+    <joint name="chassis_support_2" type="fixed">
+            <parent link="chassis"/>
+            <child link="support_2"/>
+            <origin xyz=" ${-0.3 + (0.05/2.0)} ${0.2 - (0.05/2.0)} 0.2" rpy="0 0 0"/>
+    </joint>
+    <xacro:support_link suffix = "3"/>
+    <joint name="chassis_support_3" type="fixed">
+            <parent link="chassis"/>
+            <child link="support_3"/>
+            <origin xyz=" ${-0.3 + (0.05/2.0)} ${-0.2 + (0.05/2.0)} 0.2" rpy="0 0 0"/>
+    </joint>
+    <xacro:support_link suffix = "4"/>
+    <joint name="chassis_support_4" type="fixed">
+            <parent link="chassis"/>
+            <child link="support_4"/>
+            <origin xyz=" ${0.3 - (0.05/2.0)} ${-0.2 + (0.05/2.0)} 0.2" rpy="0 0 0"/>
+    </joint>
     <joint name="base_footprint_base_joint" type="fixed">
-        <parent link="base_footprint" />
-        <child link="base_link" />
+        <parent link="base_link" />
+        <child link="chassis" />
         <origin xyz="0 0 ${wheel_radius}" rpy="0 0 0" />
     </joint>
+    <joint name="laser_base_joint" type="fixed">
+        <parent link="chassis"/>
+        <child link="laser_base_link"/>
+        <origin xyz=" 0 0 0.2" rpy="0 0 0"/>
+    </joint>
     <joint name="right_wheel_joint" type="continuous">
-        <parent link="base_link" />
+        <parent link="chassis" />
         <child link="right_wheel_link" />
         <origin xyz="${-base_length / 4.0} ${(-base_width / 2.0) - (wheel_length / 2.0) } 0" rpy="0 0 0" />
@@ -75,5 +147,5 @@
     </joint>
     <joint name="left_wheel_joint" type="continuous">
-        <parent link="base_link" />
+        <parent link="chassis" />
         <child link="left_wheel_link" />
         <origin xyz="${-base_length / 4.0} ${(base_width / 2.0) + (wheel_length / 2.0) } 0" rpy="0 0 0" />
@@ -81,5 +153,5 @@
     </joint>
     <joint name="base_caster_wheel_joint" type="fixed">
-        <parent link="base_link" />
+        <parent link="chassis" />
         <child link="caster_wheel_link" />
         <origin xyz="${base_length / 3.0} 0 ${-caster_wheel_radius}" rpy="0 0 0" />

File: diffdrive_bot/description/urdf/mira_gazebo.urdf.xacro (robot description, xacro)
@@ -5,6 +5,6 @@
     <xacro:include filename="mira_base.xacro" />
     <!-- Import bot Gazebo_ros2_control description -->
-    <xacro:include filename="lidar.xacro"/>
-    <!-- <xacro:include filename="mira_gazebo.xacro" /> -->
+    <!-- <xacro:include filename="lidar.xacro"/>
+    <xacro:include filename="mira_gazebo.xacro" /> -->
     <!-- Import bot ros2_control description -->
     <xacro:include filename="$(find diffdrive_bot)/ros2_control/diffbot.ros2_control.xacro" />

File: diffdrive_bot/description/urdf/mira_gazebo.xacro (robot description, xacro)
@@ -1,18 +1,46 @@
 <?xml version="1.0"?>
 <robot xmlns:xacro="http://www.ros.org/wiki/xacro">
-    <gazebo reference="base_link">
-        <material>Gazebo/Blue</material>
-    </gazebo>
-    <gazebo reference="right_wheel_link">
-        <material>Gazebo/Grey</material>
-    </gazebo>
-    <gazebo reference="left_wheel_link">
-        <material>Gazebo/Grey</material>
-    </gazebo>
-    <gazebo reference="caster_wheel_link">
-        <material>Gazebo/Grey</material>
-        <mu1 value="0.001" />
-        <mu2 value="0.001" />
-    </gazebo>
+  <gazebo reference="base_link">
+      <material>Gazebo/Blue</material>
+  </gazebo>
+  <gazebo reference="right_wheel_link">
+      <material>Gazebo/Grey</material>
+  </gazebo>
+  <gazebo reference="left_wheel_link">
+      <material>Gazebo/Grey</material>
+  </gazebo>
+  <gazebo reference="caster_wheel_link">
+      <material>Gazebo/Grey</material>
+      <mu1 value="0.001" />
+      <mu2 value="0.001" />
+  </gazebo>
+  <gazebo reference="laser_link">
+    <material>Gazebo/Red</material>
+    <sensor name="laser" type="ray">
+        <pose> 0 0 0 0 0 0 </pose>
+        <visualize>true</visualize>
+        <update_rate>10</update_rate>
+        <ray>
+            <scan>
+                <horizontal>
+                    <samples>360</samples>
+                    <min_angle>-3.14</min_angle>
+                    <max_angle>3.14</max_angle>
+                </horizontal>
+            </scan>
+            <range>
+                <min>0.1</min>
+                <max>10</max>
+            </range>
+        </ray>
+        <plugin name="laser_controller" filename="libgazebo_ros_ray_sensor.so">
+            <ros>
+                <argument>~/out:=raw_scan</argument>
+            </ros>
+            <output_type>sensor_msgs/LaserScan</output_type>
+            <frame_name>laser_link</frame_name>
+        </plugin>
+      </sensor>
+  </gazebo>
 <!-- ros2 control plugin -->
 <ros2_control name="GazeboSimSystem" type="system">
