Commit message: modified:   diffdrive_bot/bringup/launch/gazebo.launch.py 	renamed:    diffdrive_bot/description/urdf/mira_gazebo.xacro -> diffdrive_bot/description/urdf/gazebo.xacro 	modified:   diffdrive_bot/description/urdf/lidar.xacro 	modified:   diffdrive_bot/description/urdf/mira.urdf.xacro 	modified:   diffdrive_bot/description/urdf/mira_base.xacro 	new file:   diffdrive_bot/description/urdf/mira_gazebo.urdf.xacro 	modified:   sensor_manip/src/scan_update.cpp

File: diffdrive_bot/description/urdf/gazebo.xacro (robot description, xacro)
@@ -1,20 +1,20 @@
 <?xml version="1.0"?>
 <robot xmlns:xacro="http://www.ros.org/wiki/xacro">
-    <gazebo reference="base_link">
-        <material>Gazebo/Blue</material>
-    </gazebo>
-    <gazebo reference="right_wheel_link">
-        <material>Gazebo/Grey</material>
-    </gazebo>
-    <gazebo reference="left_wheel_link">
-        <material>Gazebo/Grey</material>
-    </gazebo>
-    <gazebo reference="caster_wheel_link">
-        <material>Gazebo/Grey</material>
-        <mu1 value="0.001" />
-        <mu2 value="0.001" />
-    </gazebo>
-<!-- ros2 control plugin -->
-<ros2_control name="GazeboSimSystem" type="system">
+  <gazebo reference="chassis">
+      <material>Gazebo/Orange</material>
+  </gazebo>
+  <gazebo reference="right_wheel_link">
+      <material>Gazebo/Grey</material>
+  </gazebo>
+  <gazebo reference="left_wheel_link">
+      <material>Gazebo/Grey</material>
+  </gazebo>
+  <gazebo reference="caster_wheel_link">
+      <material>Gazebo/Grey</material>
+      <mu1 value="0.001" />
+      <mu2 value="0.001" />
+  </gazebo>
+  <!-- ros2 control plugin -->
+  <ros2_control name="GazeboSimSystem" type="system">
     <hardware>
         <plugin>gazebo_ros2_control/GazeboSystem</plugin>

File: diffdrive_bot/description/urdf/lidar.xacro (robot description, xacro)
@@ -3,8 +3,8 @@
     <joint name="laser_joint" type="fixed">
         <parent link="laser_base_link"/>
-        <child link="laser_link"/>
-        <origin xyz=" 0 0 0.05" rpy="0 0 0"/>
+        <child link="scanner_link"/>
+        <origin xyz=" 0 0 0.01" rpy="0 0 0"/>
     </joint>
-    <link name="laser_link">
+    <link name="scanner_link">
         <visual>
             <geometry>
@@ -23,31 +23,31 @@
         </collision>
     </link>
-    <gazebo reference="laser_link">
-        <material>Gazebo/Red</material>
-        <sensor name="laser" type="ray">
-            <pose> 0 0 0 0 0 0 </pose>
-            <visualize>true</visualize>
-            <update_rate>10</update_rate>
-            <ray>
-                <scan>
-                    <horizontal>
-                        <samples>360</samples>
-                        <min_angle>-3.14</min_angle>
-                        <max_angle>3.14</max_angle>
-                    </horizontal>
-                </scan>
-                <range>
-                    <min>0.1</min>
-                    <max>10</max>
-                </range>
-            </ray>
-            <plugin name="laser_controller" filename="libgazebo_ros_ray_sensor.so">
-                <ros>
-                    <argument>~/out:=raw_scan</argument>
-                </ros>
-                <output_type>sensor_msgs/LaserScan</output_type>
-                <frame_name>laser_link</frame_name>
-            </plugin>
-        </sensor>
-    </gazebo>
+    <gazebo reference="scanner_link">
+      <material>Gazebo/Red</material>
+      <sensor name="laser" type="ray">
+          <pose> 0 0 0 0 0 0 </pose>
+          <visualize>true</visualize>
+          <update_rate>10</update_rate>
+          <ray>
+              <scan>
+                  <horizontal>
+                      <samples>360</samples>
+                      <min_angle>-3.14</min_angle>
+                      <max_angle>3.14</max_angle>
+                  </horizontal>
+              </scan>
+              <range>
+                  <min>0.1</min>
+                  <max>10</max>
+              </range>
+          </ray>
+          <plugin name="laser_controller" filename="libgazebo_ros_ray_sensor.so">
+              <ros>
+                  <argument>~/out:=raw_scan</argument>
+              </ros>
+              <output_type>sensor_msgs/LaserScan</output_type>
+              <frame_name>scanner_link</frame_name>
+          </plugin>
+      </sensor>
+  </gazebo>
 </robot>

File: diffdrive_bot/description/urdf/mira_base.xacro (robot description, xacro)
@@ -1,10 +1,12 @@
 <?xml version="1.0"?>
 <robot xmlns:xacro="http://www.ros.org/wiki/xacro">
-    <xacro:property name="base_length" value="0.6" />
-    <xacro:property name="base_width" value="0.4" />
-    <xacro:property name="base_height" value="0.2" />
-    <xacro:property name="wheel_radius" value="0.1" />
+    <xacro:property name="base_length" value="0.78" />
+    <xacro:property name="base_width" value="0.57" />
+    <xacro:property name="base_height" value="0.175" />
+    <xacro:property name="wheel_radius" value="0.075" />
     <xacro:property name="wheel_length" value="0.05" />
     <xacro:property name="caster_wheel_radius" value="${wheel_radius / 2.0}" />
+    <xacro:property name="support_side" value="0.03" />
+    <xacro:property name="support_length" value="0.15" />
     <link name="base_link" />
     <link name="base_footprint">
@@ -32,21 +34,9 @@
                            xyz="0 0 ${base_height / 2.0}" rpy="0 0 0" />
     </link>
-    <link name="laser_base_link">
-        <visual>
-            <geometry>
-                <cylinder radius="0.05" length="0.05" />
-            </geometry>
-            <origin xyz="0 0 0.025" rpy="0 0 0" />
-            <material name="blue" />
-        </visual>
-        <collision>
-            <geometry>
-                <cylinder radius="0.05" length="0.05" />
-            </geometry>
-            <origin xyz="0 0 0.025" rpy="0 0 0" />
-            <xacro:cylinder_inertia m="0.1" r="0.05" l="0.1"
-                                    xyz="0 0 0" rpy="${pi / 2.0} 0 0" />
-        </collision>
-    </link>
+    <joint name="base_link_chassis_joint" type="fixed">
+        <parent link="base_link" />
+        <child link="chassis" />
+        <origin xyz="0 0 ${wheel_radius}" rpy="0 0 0" />
+    </joint>
     <xacro:macro name="wheel_link" params="prefix">
         <link name="${prefix}_wheel_link">
@@ -69,5 +59,17 @@
     </xacro:macro>
     <xacro:wheel_link prefix="right" />
+    <joint name="right_wheel_joint" type="continuous">
+        <parent link="chassis" />
+        <child link="right_wheel_link" />
+        <origin xyz="${-base_length / 4.0} ${(-base_width / 2.0) - (wheel_length / 2.0) } 0" rpy="0 0 0" />
+        <axis xyz="0 1 0" />
+    </joint>
     <xacro:wheel_link prefix="left" />
+    <joint name="left_wheel_joint" type="continuous">
+        <parent link="chassis" />
+        <child link="left_wheel_link" />
+        <origin xyz="${-base_length / 4.0} ${(base_width / 2.0) + (wheel_length / 2.0) } 0" rpy="0 0 0" />
+        <axis xyz="0 1 0" />
+    </joint>
     <link name="caster_wheel_link">
         <visual>
@@ -87,21 +89,26 @@
                               xyz="0 0 0" rpy="0 0 0" />
     </link>
+    <joint name="chassis_caster_wheel_joint" type="fixed">
+        <parent link="chassis" />
+        <child link="caster_wheel_link" />
+        <origin xyz="${base_length / 3.0} 0 ${-caster_wheel_radius}" rpy="0 0 0" />
+    </joint>
     <xacro:macro name="support_link" params="suffix">
         <link name="support_${suffix}">
             <visual>
                 <geometry>
-                    <box size="0.05 0.05 0.2" />
+                    <box size="${support_side} ${support_side} ${support_length}" />
                 </geometry>
-                <origin xyz="0 0 0.1" rpy="0 0 0" />
+                <origin xyz="0 0 ${(support_length/2.0)}" rpy="0 0 0" />
                 <material name="blue" />
             </visual>
             <collision>
                 <geometry>
-                    <box size="0.05 0.05 0.2" />
+                    <box size="${support_side} ${support_side} ${support_length}" />
                 </geometry>
-                <origin xyz="0 0 0.1" rpy="0 0 0" />
+                <origin xyz="0 0 ${(support_length/2.0)}" rpy="0 0 0" />
             </collision>
-            <xacro:box_inertia m="1.0" l="${2*0.05}" w="${2*0.05}" h="${2*0.2}"
-                            xyz="0 0 0.1" rpy="0 0 0" />
+            <xacro:box_inertia m="1.0" l="${2*support_side}" w="${2*support_side}" h="${2*support_length}"
+                            xyz="0 0 ${(support_length/2.0)}" rpy="0 0 0" />
         </link>
     </xacro:macro>
@@ -110,5 +117,5 @@
             <parent link="chassis"/>
             <child link="support_1"/>
-            <origin xyz=" ${0.3 - (0.05/2.0)} ${0.2 - (0.05/2.0)} 0.2" rpy="0 0 0"/>
+            <origin xyz=" ${(base_length/2.0) - (support_side/2.0)} ${(base_width/2.0) - (support_side/2.0)} ${base_height}" rpy="0 0 0"/>
     </joint>
     <xacro:support_link suffix = "2"/>
@@ -116,5 +123,5 @@
             <parent link="chassis"/>
             <child link="support_2"/>
-            <origin xyz=" ${-0.3 + (0.05/2.0)} ${0.2 - (0.05/2.0)} 0.2" rpy="0 0 0"/>
+            <origin xyz=" 0.0 ${(base_width/2.0) - (support_side/2.0)} ${base_height}" rpy="0 0 0"/>
     </joint>
     <xacro:support_link suffix = "3"/>
@@ -122,5 +129,5 @@
             <parent link="chassis"/>
             <child link="support_3"/>
-            <origin xyz=" ${-0.3 + (0.05/2.0)} ${-0.2 + (0.05/2.0)} 0.2" rpy="0 0 0"/>
+            <origin xyz=" ${-(base_length/2.0) + (support_side/2.0)} ${(base_width/2.0) - (support_side/2.0)} ${base_height}" rpy="0 0 0"/>
     </joint>
     <xacro:support_link suffix = "4"/>
@@ -128,32 +135,39 @@
             <parent link="chassis"/>
             <child link="support_4"/>
-            <origin xyz=" ${0.3 - (0.05/2.0)} ${-0.2 + (0.05/2.0)} 0.2" rpy="0 0 0"/>
+            <origin xyz=" ${-(base_length/2.0) + (support_side/2.0)} ${-(base_width/2.0) + (support_side/2.0)} ${base_height}" rpy="0 0 0"/>
     </joint>
-    <joint name="base_footprint_base_joint" type="fixed">
-        <parent link="base_link" />
-        <child link="chassis" />
-        <origin xyz="0 0 ${wheel_radius}" rpy="0 0 0" />
+    <xacro:support_link suffix = "5"/>
+    <joint name="chassis_support_5" type="fixed">
+            <parent link="chassis"/>
+            <child link="support_5"/>
+            <origin xyz=" 0.0 ${-(base_width/2.0) + (support_side/2.0)} ${base_height}" rpy="0 0 0"/>
     </joint>
-    <joint name="laser_base_joint" type="fixed">
+    <xacro:support_link suffix = "6"/>
+    <joint name="chassis_support_6" type="fixed">
+            <parent link="chassis"/>
+            <child link="support_6"/>
+            <origin xyz=" ${(base_length/2.0) - (support_side/2.0)} ${-(base_width/2.0) + (support_side/2.0)} ${base_height}" rpy="0 0 0"/>
+    </joint>
+    <link name="laser_base_link">
+        <visual>
+            <geometry>
+                <cylinder radius="0.05" length="0.01" />
+            </geometry>
+            <origin xyz="0 0 0.0" rpy="0 0 0" />
+            <material name="blue" />
+        </visual>
+        <collision>
+            <geometry>
+                <cylinder radius="0.05" length="0.01" />
+            </geometry>
+            <origin xyz="0 0 0" rpy="0 0 0" />
+            <xacro:cylinder_inertia m="0.1" r="0.05" l="0.1"
+                                    xyz="0 0 0" rpy="${pi / 2.0} 0 0" />
+        </collision>
+    </link>
+    <joint name="chassis_laser_base_joint" type="fixed">
         <parent link="chassis"/>
         <child link="laser_base_link"/>
-        <origin xyz=" 0 0 0.2" rpy="0 0 0"/>
-    </joint>
-    <joint name="right_wheel_joint" type="continuous">
-        <parent link="chassis" />
-        <child link="right_wheel_link" />
-        <origin xyz="${-base_length / 4.0} ${(-base_width / 2.0) - (wheel_length / 2.0) } 0" rpy="0 0 0" />
-        <axis xyz="0 1 0" />
-    </joint>
-    <joint name="left_wheel_joint" type="continuous">
-        <parent link="chassis" />
-        <child link="left_wheel_link" />
-        <origin xyz="${-base_length / 4.0} ${(base_width / 2.0) + (wheel_length / 2.0) } 0" rpy="0 0 0" />
-        <axis xyz="0 1 0" />
-    </joint>
-    <joint name="base_caster_wheel_joint" type="fixed">
-        <parent link="chassis" />
-        <child link="caster_wheel_link" />
-        <origin xyz="${base_length / 3.0} 0 ${-caster_wheel_radius}" rpy="0 0 0" />
+        <origin xyz=" ${(base_length/2.0)-(0.05)} 0 ${base_height}" rpy="0 0 0"/>
     </joint>
 </robot>

File: diffdrive_bot/description/urdf/mira_gazebo.urdf.xacro (robot description, xacro)
@@ -6,7 +6,5 @@
     <!-- Import bot Gazebo_ros2_control description -->
     <xacro:include filename="lidar.xacro"/>
-    <!-- Import bot ros2_control description -->
-    <xacro:include filename="$(find diffdrive_bot)/ros2_control/diffbot.ros2_control.xacro" />
-    <xacro:bot_ros2_control name="mira" prefix="$(arg prefix)" />
+    <xacro:include filename="gazebo.xacro" />
     <!-- <xacro:include filename="camera.xacro" /> -->
 </robot>
