Commit message: modified:   diffdrive_bot/bringup/launch/rviz.launch.xml 	new file:   diffdrive_bot/description/rviz/mira.rviz 	modified:   diffdrive_bot/description/urdf/lidar.xacro 	modified:   diffdrive_bot/description/urdf/mira_base.xacro

File: diffdrive_bot/description/urdf/lidar.xacro (robot description, xacro)
@@ -38,5 +38,5 @@
                 </scan>
                 <range>
-                    <min>0.5</min>
+                    <min>0.1</min>
                     <max>10</max>
                 </range>

File: diffdrive_bot/description/urdf/mira_base.xacro (robot description, xacro)
@@ -87,4 +87,47 @@
                               xyz="0 0 0" rpy="0 0 0" />
     </link>
+    <xacro:macro name="support_link" params="suffix">
+        <link name="support_${suffix}">
+            <visual>
+                <geometry>
+                    <box size="0.05 0.05 0.2" />
+                </geometry>
+                <origin xyz="0 0 0.1" rpy="0 0 0" />
+                <material name="blue" />
+            </visual>
+            <collision>
+                <geometry>
+                    <box size="0.05 0.05 0.2" />
+                </geometry>
+                <origin xyz="0 0 0.1" rpy="0 0 0" />
+            </collision>
+            <xacro:box_inertia m="1.0" l="${2*0.05}" w="${2*0.05}" h="${2*0.2}"
+                            xyz="0 0 0.1" rpy="0 0 0" />
+        </link>
+    </xacro:macro>
+    <xacro:support_link suffix = "1"/>
+    <joint name="chassis_support_1" type="fixed">
+            <parent link="chassis"/>
+            <child link="support_1"/>
+            <origin xyz=" ${0.3 - (0.05/2.0)} ${0.2 - (0.05/2.0)} 0.2" rpy="0 0 0"/>
+    </joint>
+    <xacro:support_link suffix = "2"/>
+    <joint name="chassis_support_2" type="fixed">
+            <parent link="chassis"/>
+            <child link="support_2"/>
+            <origin xyz=" ${-0.3 + (0.05/2.0)} ${0.2 - (0.05/2.0)} 0.2" rpy="0 0 0"/>
+    </joint>
+    <xacro:support_link suffix = "3"/>
+    <joint name="chassis_support_3" type="fixed">
+            <parent link="chassis"/>
+            <child link="support_3"/>
+            <origin xyz=" ${-0.3 + (0.05/2.0)} ${-0.2 + (0.05/2.0)} 0.2" rpy="0 0 0"/>
+    </joint>
+    <xacro:support_link suffix = "4"/>
+    <joint name="chassis_support_4" type="fixed">
+            <parent link="chassis"/>
+            <child link="support_4"/>
+            <origin xyz=" ${0.3 - (0.05/2.0)} ${-0.2 + (0.05/2.0)} 0.2" rpy="0 0 0"/>
+    </joint>
     <joint name="base_footprint_base_joint" type="fixed">
         <parent link="base_link" />

Commit message: new file:   .vscode/c_cpp_properties.json 	new file:   .vscode/settings.json 	modified:   diffdrive_bot/bringup/launch/gazebo.launch.py 	modified:   diffdrive_bot/description/urdf/lidar.xacro 	modified:   diffdrive_bot/description/urdf/mira_base.xacro 	modified:   diffdrive_bot/description/urdf/mira_gazebo.urdf.xacro 	modified:   diffdrive_bot/description/urdf/mira_gazebo.xacro 	modified:   sensor_manip/src/scan_update.cpp

File: diffdrive_bot/description/urdf/lidar.xacro (robot description, xacro)
@@ -1,12 +1,12 @@
 <?xml version="1.0"?>
 <robot xmlns:xacro="http://www.ros.org/wiki/xacro">
-    <xacro:include filename="$(find pf_description)/urdf/r2000.urdf.xacro" />
-    <xacro:r2000 prefix="" />
+    <!-- <xacro:include filename="$(find pf_description)/urdf/r2000.urdf.xacro" />
+    <xacro:r2000 prefix="" /> -->
     <joint name="laser_joint" type="fixed">
         <parent link="laser_base_link"/>
         <child link="scanner_link"/>
-        <origin xyz=" 0 0 0.05" rpy="0 0 0"/>
+        <origin xyz=" 0 0 0.01" rpy="0 0 0"/>
     </joint>
-    <!-- <link name="scanner_link">
+    <link name="scanner_link">
         <visual>
             <geometry>
@@ -24,4 +24,4 @@
                                     xyz="0 0 0" rpy="${pi / 2.0} 0 0" />
         </collision>
-    </link> -->
+    </link>
 </robot>

File: diffdrive_bot/description/urdf/mira_base.xacro (robot description, xacro)
@@ -1,8 +1,8 @@
 <?xml version="1.0"?>
 <robot xmlns:xacro="http://www.ros.org/wiki/xacro">
-    <xacro:property name="base_length" value="0.6" />
-    <xacro:property name="base_width" value="0.4" />
-    <xacro:property name="base_height" value="0.2" />
-    <xacro:property name="wheel_radius" value="0.1" />
+    <xacro:property name="base_length" value="0.78" />
+    <xacro:property name="base_width" value="0.57" />
+    <xacro:property name="base_height" value="0.175" />
+    <xacro:property name="wheel_radius" value="0.075" />
     <xacro:property name="wheel_length" value="0.05" />
     <xacro:property name="caster_wheel_radius" value="${wheel_radius / 2.0}" />
@@ -35,14 +35,14 @@
         <visual>
             <geometry>
-                <cylinder radius="0.05" length="0.05" />
+                <cylinder radius="0.05" length="0.01" />
             </geometry>
-            <origin xyz="0 0 0.025" rpy="0 0 0" />
+            <origin xyz="0 0 0" rpy="0 0 0" />
             <material name="blue" />
         </visual>
         <collision>
             <geometry>
-                <cylinder radius="0.05" length="0.05" />
+                <cylinder radius="0.05" length="0.01" />
             </geometry>
-            <origin xyz="0 0 0.025" rpy="0 0 0" />
+            <origin xyz="0 0 0" rpy="0 0 0" />
             <xacro:cylinder_inertia m="0.1" r="0.05" l="0.1"
                                     xyz="0 0 0" rpy="${pi / 2.0} 0 0" />
@@ -91,17 +91,17 @@
             <visual>
                 <geometry>
-                    <box size="0.05 0.05 0.2" />
+                    <box size="0.03 0.03 0.15" />
                 </geometry>
-                <origin xyz="0 0 0.1" rpy="0 0 0" />
+                <origin xyz="0 0 0.075" rpy="0 0 0" />
                 <material name="blue" />
             </visual>
             <collision>
                 <geometry>
-                    <box size="0.05 0.05 0.2" />
+                    <box size="0.03 0.03 0.15" />
                 </geometry>
-                <origin xyz="0 0 0.1" rpy="0 0 0" />
+                <origin xyz="0 0 0.075" rpy="0 0 0" />
             </collision>
-            <xacro:box_inertia m="1.0" l="${2*0.05}" w="${2*0.05}" h="${2*0.2}"
-                            xyz="0 0 0.1" rpy="0 0 0" />
+            <xacro:box_inertia m="1.0" l="${2*0.03}" w="${2*0.03}" h="${2*0.15}"
+                            xyz="0 0 0.075" rpy="0 0 0" />
         </link>
     </xacro:macro>
@@ -110,5 +110,5 @@
             <parent link="chassis"/>
             <child link="support_1"/>
-            <origin xyz=" ${0.3 - (0.05/2.0)} ${0.2 - (0.05/2.0)} 0.2" rpy="0 0 0"/>
+            <origin xyz=" ${(0.78/2.0) - (0.03/2.0)} ${(0.57/2.0) - (0.03/2.0)} ${base_height}" rpy="0 0 0"/>
     </joint>
     <xacro:support_link suffix = "2"/>
@@ -116,5 +116,5 @@
             <parent link="chassis"/>
             <child link="support_2"/>
-            <origin xyz=" ${-0.3 + (0.05/2.0)} ${0.2 - (0.05/2.0)} 0.2" rpy="0 0 0"/>
+            <origin xyz=" 0.0 ${(0.57/2.0) - (0.03/2.0)} ${base_height}" rpy="0 0 0"/>
     </joint>
     <xacro:support_link suffix = "3"/>
@@ -122,5 +122,5 @@
             <parent link="chassis"/>
             <child link="support_3"/>
-            <origin xyz=" ${-0.3 + (0.05/2.0)} ${-0.2 + (0.05/2.0)} 0.2" rpy="0 0 0"/>
+            <origin xyz=" ${-(0.78/2.0) + (0.03/2.0)} ${(0.57/2.0) - (0.03/2.0)} ${base_height}" rpy="0 0 0"/>
     </joint>
     <xacro:support_link suffix = "4"/>
@@ -128,5 +128,17 @@
             <parent link="chassis"/>
             <child link="support_4"/>
-            <origin xyz=" ${0.3 - (0.05/2.0)} ${-0.2 + (0.05/2.0)} 0.2" rpy="0 0 0"/>
+            <origin xyz=" ${-(0.78/2.0) + (0.03/2.0)} ${-(0.57/2.0) + (0.03/2.0)} ${base_height}" rpy="0 0 0"/>
+    </joint>
+    <xacro:support_link suffix = "5"/>
+    <joint name="chassis_support_5" type="fixed">
+            <parent link="chassis"/>
+            <child link="support_5"/>
+            <origin xyz=" 0.0 ${-(0.57/2.0) + (0.03/2.0)} ${base_height}" rpy="0 0 0"/>
+    </joint>
+    <xacro:support_link suffix = "6"/>
+    <joint name="chassis_support_6" type="fixed">
+            <parent link="chassis"/>
+            <child link="support_6"/>
+            <origin xyz=" ${(0.78/2.0) - (0.03/2.0)} ${-(0.57/2.0) + (0.03/2.0)} ${base_height}" rpy="0 0 0"/>
     </joint>
     <joint name="base_footprint_base_joint" type="fixed">
@@ -138,5 +150,5 @@
         <parent link="chassis"/>
         <child link="laser_base_link"/>
-        <origin xyz=" 0 0 0.2" rpy="0 0 0"/>
+        <origin xyz="${(0.78/2.0)-(0.05 + 0.03)}  0 ${base_height}" rpy="0 0 0"/>
     </joint>
     <joint name="right_wheel_joint" type="continuous">

File: diffdrive_bot/description/urdf/mira_gazebo.urdf.xacro (robot description, xacro)
@@ -5,9 +5,9 @@
     <xacro:include filename="mira_base.xacro" />
     <!-- Import bot Gazebo_ros2_control description -->
-    <!-- <xacro:include filename="lidar.xacro"/>
-    <xacro:include filename="mira_gazebo.xacro" /> -->
+    <xacro:include filename="lidar.xacro"/>
+    <xacro:include filename="mira_gazebo.xacro" />
     <!-- Import bot ros2_control description -->
-    <xacro:include filename="$(find diffdrive_bot)/ros2_control/diffbot.ros2_control.xacro" />
-    <xacro:bot_ros2_control name="mira" prefix="$(arg prefix)" />
+    <!-- <xacro:include filename="$(find diffdrive_bot)/ros2_control/diffbot.ros2_control.xacro" />
+    <xacro:bot_ros2_control name="mira" prefix="$(arg prefix)" /> -->
     <!-- <xacro:include filename="camera.xacro" /> -->
 </robot>

File: diffdrive_bot/description/urdf/mira_gazebo.xacro (robot description, xacro)
@@ -15,5 +15,5 @@
       <mu2 value="0.001" />
   </gazebo>
-  <gazebo reference="laser_link">
+  <gazebo reference="scanner_link">
     <material>Gazebo/Red</material>
     <sensor name="laser" type="ray">
@@ -39,5 +39,5 @@
             </ros>
             <output_type>sensor_msgs/LaserScan</output_type>
-            <frame_name>laser_link</frame_name>
+            <frame_name>scanner_link</frame_name>
         </plugin>
       </sensor>

Commit message: modified:   diffdrive_bot/CMakeLists.txt 	modified:   diffdrive_bot/bringup/config/mapper_params_online_async.yaml 	modified:   diffdrive_bot/bringup/launch/custom_cartographer.launch.py 	modified:   diffdrive_bot/bringup/launch/diffbot.launch.py 	modified:   diffdrive_bot/description/urdf/lidar.xacro 	modified:   diffdrive_bot/package.xml 	modified:   sensor_manip/src/scan_update.cpp

File: diffdrive_bot/description/urdf/lidar.xacro (robot description, xacro)
@@ -1,6 +1,6 @@
 <?xml version="1.0"?>
 <robot xmlns:xacro="http://www.ros.org/wiki/xacro">
-    <!-- <xacro:include filename="$(find pf_description)/urdf/r2000.urdf.xacro" />
-    <xacro:r2000 prefix="" /> -->
+    <xacro:include filename="$(find pf_description)/urdf/r2000.urdf.xacro" />
+    <xacro:r2000 prefix="" />
     <joint name="laser_joint" type="fixed">
         <parent link="laser_base_link"/>
@@ -8,5 +8,5 @@
         <origin xyz=" 0 0 0.01" rpy="0 0 0"/>
     </joint>
-    <link name="scanner_link">
+    <!-- <link name="scanner_link">
         <visual>
             <geometry>
@@ -24,4 +24,4 @@
                                     xyz="0 0 0" rpy="${pi / 2.0} 0 0" />
         </collision>
-    </link>
+    </link> -->
 </robot>

Commit message: modified:   diffdrive_bot/bringup/config/mapper_params_online_async.yaml 	modified:   diffdrive_bot/bringup/launch/custom_cartographer.launch.py 	modified:   diffdrive_bot/bringup/launch/gazebo.launch.py 	new file:   diffdrive_bot/description/rviz/r2000.rviz 	renamed:    diffdrive_bot/description/urdf/mira_gazebo.xacro -> diffdrive_bot/description/urdf/gazebo.xacro 	modified:   diffdrive_bot/description/urdf/lidar.xacro 	modified:   diffdrive_bot/description/urdf/mira.urdf.xacro 	modified:   diffdrive_bot/description/urdf/mira_base.xacro 	modified:   diffdrive_bot/description/urdf/mira_gazebo.urdf.xacro

File: diffdrive_bot/description/urdf/lidar.xacro (robot description, xacro)
@@ -6,5 +6,5 @@
         <parent link="laser_base_link"/>
         <child link="scanner_link"/>
-        <origin xyz=" 0 0 0.01" rpy="0 0 0"/>
+        <origin xyz=" 0.0 0 0.175" rpy="0 0 0"/>
     </joint>
     <!-- <link name="scanner_link">

File: diffdrive_bot/description/urdf/mira.urdf.xacro (robot description, xacro)
@@ -6,5 +6,4 @@
     <!-- Import bot Gazebo_ros2_control description -->
     <xacro:include filename="lidar.xacro"/>
-    <!-- <xacro:include filename="mira_gazebo.xacro" /> -->
     <!-- Import bot ros2_control description -->
     <xacro:include filename="$(find diffdrive_bot)/ros2_control/diffbot.ros2_control.xacro" />

File: diffdrive_bot/description/urdf/mira_base.xacro (robot description, xacro)
@@ -7,4 +7,6 @@
     <xacro:property name="wheel_length" value="0.05" />
     <xacro:property name="caster_wheel_radius" value="${wheel_radius / 2.0}" />
+    <xacro:property name="support_side" value="0.03" />
+    <xacro:property name="support_length" value="0.15" />
     <link name="base_link" />
     <link name="base_footprint">
@@ -32,21 +34,9 @@
                            xyz="0 0 ${base_height / 2.0}" rpy="0 0 0" />
     </link>
-    <link name="laser_base_link">
-        <visual>
-            <geometry>
-                <cylinder radius="0.05" length="0.01" />
-            </geometry>
-            <origin xyz="0 0 0" rpy="0 0 0" />
-            <material name="blue" />
-        </visual>
-        <collision>
-            <geometry>
-                <cylinder radius="0.05" length="0.01" />
-            </geometry>
-            <origin xyz="0 0 0" rpy="0 0 0" />
-            <xacro:cylinder_inertia m="0.1" r="0.05" l="0.1"
-                                    xyz="0 0 0" rpy="${pi / 2.0} 0 0" />
-        </collision>
-    </link>
+    <joint name="base_link_chassis_joint" type="fixed">
+        <parent link="base_link" />
+        <child link="chassis" />
+        <origin xyz="0 0 ${wheel_radius}" rpy="0 0 0" />
+    </joint>
     <xacro:macro name="wheel_link" params="prefix">
         <link name="${prefix}_wheel_link">
@@ -69,5 +59,17 @@
     </xacro:macro>
     <xacro:wheel_link prefix="right" />
+    <joint name="right_wheel_joint" type="continuous">
+        <parent link="chassis" />
+        <child link="right_wheel_link" />
+        <origin xyz="${-base_length / 4.0} ${(-base_width / 2.0) - (wheel_length / 2.0) } 0" rpy="0 0 0" />
+        <axis xyz="0 1 0" />
+    </joint>
     <xacro:wheel_link prefix="left" />
+    <joint name="left_wheel_joint" type="continuous">
+        <parent link="chassis" />
+        <child link="left_wheel_link" />
+        <origin xyz="${-base_length / 4.0} ${(base_width / 2.0) + (wheel_length / 2.0) } 0" rpy="0 0 0" />
+        <axis xyz="0 1 0" />
+    </joint>
     <link name="caster_wheel_link">
         <visual>
@@ -87,21 +89,26 @@
                               xyz="0 0 0" rpy="0 0 0" />
     </link>
+    <joint name="chassis_caster_wheel_joint" type="fixed">
+        <parent link="chassis" />
+        <child link="caster_wheel_link" />
+        <origin xyz="${base_length / 3.0} 0 ${-caster_wheel_radius}" rpy="0 0 0" />
+    </joint>
     <xacro:macro name="support_link" params="suffix">
         <link name="support_${suffix}">
             <visual>
                 <geometry>
-                    <box size="0.03 0.03 0.15" />
+                    <box size="${support_side} ${support_side} ${support_length}" />
                 </geometry>
-                <origin xyz="0 0 0.075" rpy="0 0 0" />
+                <origin xyz="0 0 ${(support_length/2.0)}" rpy="0 0 0" />
                 <material name="blue" />
             </visual>
             <collision>
                 <geometry>
-                    <box size="0.03 0.03 0.15" />
+                    <box size="${support_side} ${support_side} ${support_length}" />
                 </geometry>
-                <origin xyz="0 0 0.075" rpy="0 0 0" />
+                <origin xyz="0 0 ${(support_length/2.0)}" rpy="0 0 0" />
             </collision>
-            <xacro:box_inertia m="1.0" l="${2*0.03}" w="${2*0.03}" h="${2*0.15}"
-                            xyz="0 0 0.075" rpy="0 0 0" />
+            <xacro:box_inertia m="1.0" l="${2*support_side}" w="${2*support_side}" h="${2*support_length}"
+                            xyz="0 0 ${(support_length/2.0)}" rpy="0 0 0" />
         </link>
     </xacro:macro>
@@ -110,5 +117,5 @@
             <parent link="chassis"/>
             <child link="support_1"/>
-            <origin xyz=" ${(0.78/2.0) - (0.03/2.0)} ${(0.57/2.0) - (0.03/2.0)} ${base_height}" rpy="0 0 0"/>
+            <origin xyz=" ${(base_length/2.0) - (support_side/2.0)} ${(base_width/2.0) - (support_side/2.0)} ${base_height}" rpy="0 0 0"/>
     </joint>
     <xacro:support_link suffix = "2"/>
@@ -116,5 +123,5 @@
             <parent link="chassis"/>
             <child link="support_2"/>
-            <origin xyz=" 0.0 ${(0.57/2.0) - (0.03/2.0)} ${base_height}" rpy="0 0 0"/>
+            <origin xyz=" 0.0 ${(base_width/2.0) - (support_side/2.0)} ${base_height}" rpy="0 0 0"/>
     </joint>
     <xacro:support_link suffix = "3"/>
@@ -122,5 +129,5 @@
             <parent link="chassis"/>
             <child link="support_3"/>
-            <origin xyz=" ${-(0.78/2.0) + (0.03/2.0)} ${(0.57/2.0) - (0.03/2.0)} ${base_height}" rpy="0 0 0"/>
+            <origin xyz=" ${-(base_length/2.0) + (support_side/2.0)} ${(base_width/2.0) - (support_side/2.0)} ${base_height}" rpy="0 0 0"/>
     </joint>
     <xacro:support_link suffix = "4"/>
@@ -128,5 +135,5 @@
             <parent link="chassis"/>
             <child link="support_4"/>
-            <origin xyz=" ${-(0.78/2.0) + (0.03/2.0)} ${-(0.57/2.0) + (0.03/2.0)} ${base_height}" rpy="0 0 0"/>
+            <origin xyz=" ${-(base_length/2.0) + (support_side/2.0)} ${-(base_width/2.0) + (support_side/2.0)} ${base_height}" rpy="0 0 0"/>
     </joint>
     <xacro:support_link suffix = "5"/>
@@ -134,5 +141,5 @@
             <parent link="chassis"/>
             <child link="support_5"/>
-            <origin xyz=" 0.0 ${-(0.57/2.0) + (0.03/2.0)} ${base_height}" rpy="0 0 0"/>
+            <origin xyz=" 0.0 ${-(base_width/2.0) + (support_side/2.0)} ${base_height}" rpy="0 0 0"/>
     </joint>
     <xacro:support_link suffix = "6"/>
@@ -140,32 +147,27 @@
             <parent link="chassis"/>
             <child link="support_6"/>
-            <origin xyz=" ${(0.78/2.0) - (0.03/2.0)} ${-(0.57/2.0) + (0.03/2.0)} ${base_height}" rpy="0 0 0"/>
+            <origin xyz=" ${(base_length/2.0) - (support_side/2.0)} ${-(base_width/2.0) + (support_side/2.0)} ${base_height}" rpy="0 0 0"/>
     </joint>
-    <joint name="base_footprint_base_joint" type="fixed">
-        <parent link="base_link" />
-        <child link="chassis" />
-        <origin xyz="0 0 ${wheel_radius}" rpy="0 0 0" />
-    </joint>
-    <joint name="laser_base_joint" type="fixed">
+    <link name="laser_base_link">
+        <visual>
+            <geometry>
+                <cylinder radius="0.05" length="0.01" />
+            </geometry>
+            <origin xyz="0 0 0.0" rpy="0 0 0" />
+            <material name="blue" />
+        </visual>
+        <collision>
+            <geometry>
+                <cylinder radius="0.05" length="0.01" />
+            </geometry>
+            <origin xyz="0 0 0" rpy="0 0 0" />
+            <xacro:cylinder_inertia m="0.1" r="0.05" l="0.1"
+                                    xyz="0 0 0" rpy="${pi / 2.0} 0 0" />
+        </collision>
+    </link>
+    <joint name="chassis_laser_base_joint" type="fixed">
         <parent link="chassis"/>
         <child link="laser_base_link"/>
-        <origin xyz="${(0.78/2.0)-(0.05 + 0.03)}  0 ${base_height}" rpy="0 0 0"/>
-    </joint>
-    <joint name="right_wheel_joint" type="continuous">
-        <parent link="chassis" />
-        <child link="right_wheel_link" />
-        <origin xyz="${-base_length / 4.0} ${(-base_width / 2.0) - (wheel_length / 2.0) } 0" rpy="0 0 0" />
-        <axis xyz="0 1 0" />
-    </joint>
-    <joint name="left_wheel_joint" type="continuous">
-        <parent link="chassis" />
-        <child link="left_wheel_link" />
-        <origin xyz="${-base_length / 4.0} ${(base_width / 2.0) + (wheel_length / 2.0) } 0" rpy="0 0 0" />
-        <axis xyz="0 1 0" />
-    </joint>
-    <joint name="base_caster_wheel_joint" type="fixed">
-        <parent link="chassis" />
-        <child link="caster_wheel_link" />
-        <origin xyz="${base_length / 3.0} 0 ${-caster_wheel_radius}" rpy="0 0 0" />
+        <origin xyz=" ${(base_length/2.0)-(0.05)} 0 ${base_height}" rpy="0 0 0"/>
     </joint>
 </robot>

File: diffdrive_bot/description/urdf/mira_gazebo.urdf.xacro (robot description, xacro)
@@ -6,8 +6,5 @@
     <!-- Import bot Gazebo_ros2_control description -->
     <xacro:include filename="lidar.xacro"/>
-    <xacro:include filename="mira_gazebo.xacro" />
-    <!-- Import bot ros2_control description -->
-    <!-- <xacro:include filename="$(find diffdrive_bot)/ros2_control/diffbot.ros2_control.xacro" />
-    <xacro:bot_ros2_control name="mira" prefix="$(arg prefix)" /> -->
+    <xacro:include filename="gazebo.xacro" />
     <!-- <xacro:include filename="camera.xacro" /> -->
 </robot>

Commit message: modified:   diffdrive_bot/bringup/config/mira_controller.yaml 	modified:   diffdrive_bot/description/urdf/lidar.xacro 	modified:   diffdrive_bot/hardware/include/diffdrive_bot/motor_handler.hpp 	modified:   diffdrive_bot/hardware/src/motor_handler.cpp

File: diffdrive_bot/description/urdf/lidar.xacro (robot description, xacro)
@@ -4,5 +4,5 @@
     <xacro:r2000 prefix="" />
     <joint name="laser_joint" type="fixed">
-        <parent link="base_footprint"/>
+        <parent link="laser_base_link"/>
         <child link="scanner_link"/>
         <origin xyz=" 0.0 0 0.110" rpy="0 0 0"/>
