Commit message: modified:   .vscode/c_cpp_properties.json 	modified:   diffdrive_bot/bringup/config/mapper_params_online_async.yaml 	modified:   diffdrive_bot/bringup/config/mira_controller.yaml 	modified:   diffdrive_bot/bringup/launch/custom_cartographer.launch.py 	modified:   diffdrive_bot/bringup/launch/diffbot.launch.py 	modified:   diffdrive_bot/description/ros2_control/diffbot.ros2_control.xacro 	modified:   diffdrive_bot/description/rviz/r2000.rviz 	modified:   diffdrive_bot/description/urdf/lidar.xacro 	modified:   diffdrive_bot/description/urdf/mira_base.xacro 	modified:   diffdrive_bot/hardware/src/motor_handler.cpp

File: diffdrive_bot/description/ros2_control/diffbot.ros2_control.xacro (robot description, xacro)
@@ -7,5 +7,5 @@
         <param name="l_drive_name">left_wheel_joint</param>
         <param name="l_serial_port">/dev/ttyACM0</param>
-        <param name="l_baud">9600</param>
+        <param name="l_baud">57600</param>
         <param name="l_stop_bit">1</param>
         <param name="l_data_bit">8</param>
@@ -15,5 +15,5 @@
         <param name="r_drive_name">right_wheel_joint</param>
         <param name="r_serial_port">/dev/ttyACM0</param>
-        <param name="r_baud">9600</param>
+        <param name="r_baud">57600</param>
         <param name="r_stop_bit">1</param>
         <param name="r_data_bit">8</param>

File: diffdrive_bot/description/urdf/lidar.xacro (robot description, xacro)
@@ -4,7 +4,7 @@
     <xacro:r2000 prefix="" />
     <joint name="laser_joint" type="fixed">
-        <parent link="laser_base_link"/>
+        <parent link="base_footprint"/>
         <child link="scanner_link"/>
-        <origin xyz=" 0.0 0 0.175" rpy="0 0 0"/>
+        <origin xyz=" 0.0 0 0.110" rpy="0 0 0"/>
     </joint>
     <!-- <link name="scanner_link">

File: diffdrive_bot/description/urdf/mira_base.xacro (robot description, xacro)
@@ -169,5 +169,5 @@
         <parent link="chassis"/>
         <child link="laser_base_link"/>
-        <origin xyz=" ${(base_length/2.0)-(0.05)} 0 ${base_height}" rpy="0 0 0"/>
+        <origin xyz=" ${(base_length/2.0)-(0.05+0.03)} 0 ${base_height}" rpy="0 0 0"/>
     </joint>
 </robot>
